Commit message: navigation progress and add executable

File: description/lidar.xacro (robot description, xacro)
@@ -4,5 +4,5 @@
         <parent link="chassis"/>
         <child link="laser_frame"/>
-        <origin xyz="0.3769 0 0.212" rpy="0 0 0"/>
+        <origin xyz="0.7219 0.0005 0.232" rpy="0 0 1.5708"/>
     </joint>
     <link name="laser_frame">

File: description/robot.urdf.xacro (robot description, xacro)
@@ -13,4 +13,4 @@
     <xacro:include filename="lidar.xacro" />
     <!-- <xacro:include filename="camera.xacro" /> -->
-    <xacro:include filename="face.xacro" />
+    <!-- <xacro:include filename="face.xacro" /> -->
 </robot>
